File: More/hardware/boards/HEGduinoV1/HEG_Sensor.brd (EAGLE design)
At the start: 166 x 25.4 mm, 17 parts, among them J1 A-2004-1-4-LP-N-R

Commit message: Added some sensor designs, moved some stuff
Other:
- outline, holes or cut-outs redrawn
- board text added: "By Joshua Brewster (MIT License) Inspired by patent 5995857"
Changed lines of the file:
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@@
 <circle x="98.58375" y="25.7175" radius="0.502009375" width="0.1016" layer="101"/>
 <circle x="101.12375" y="25.7175" radius="0.502009375" width="0.1016" layer="101"/>
+<text x="133.35" y="19.84375" size="1.778" layer="25">By Joshua Brewster (MIT License)
+Inspired by patent 5995857</text>
+<wire x1="182.40375" y1="22.5425" x2="182.40375" y2="37.30625" width="0.1524" layer="20"/>
+<wire x1="182.40375" y1="37.30625" x2="182.72125" y2="37.62375" width="0.1524" layer="20" curve="-90"/>
+<wire x1="182.72125" y1="37.62375" x2="183.67375" y2="37.62375" width="0.1524" layer="20"/>
+<wire x1="183.67375" y1="37.62375" x2="183.99125" y2="37.30625" width="0.1524" layer="20" curve="-90"/>
+<wire x1="183.99125" y1="37.30625" x2="183.99125" y2="22.5425" width="0.1524" layer="20"/>
+<wire x1="183.99125" y1="22.5425" x2="183.67375" y2="22.225" width="0.1524" layer="20" curve="-90"/>
+<wire x1="183.67375" y1="22.225" x2="182.72125" y2="22.225" width="0.1524" layer="20"/>
+<wire x1="182.72125" y1="22.225" x2="182.40375" y2="22.5425" width="0.1524" layer="20" curve="-90"/>
+<wire x1="182.40375" y1="22.5425" x2="182.40375" y2="37.30625" width="0.1524" layer="101"/>
+<wire x1="182.40375" y1="37.30625" x2="182.72125" y2="37.62375" width="0.1524" layer="101" curve="-90"/>
+<wire x1="182.72125" y1="37.62375" x2="183.67375" y2="37.62375" width="0.1524" layer="101"/>
+<wire x1="183.67375" y1="37.62375" x2="183.99125" y2="37.30625" width="0.1524" layer="101" curve="-90"/>
+<wire x1="183.99125" y1="37.30625" x2="183.99125" y2="22.5425" width="0.1524" layer="101"/>
+<wire x1="183.99125" y1="22.5425" x2="183.67375" y2="22.225" width="0.1524" layer="101" curve="-90"/>
+<wire x1="183.67375" y1="22.225" x2="182.72125" y2="22.225" width="0.1524" layer="101"/>
+<wire x1="182.72125" y1="22.225" x2="182.40375" y2="22.5425" width="0.1524" layer="101" curve="-90"/>
+<wire x1="182.40375" y1="22.5425" x2="182.40375" y2="37.30625" width="0.1524" layer="100"/>
+<wire x1="182.40375" y1="37.30625" x2="182.72125" y2="37.62375" width="0.1524" layer="100" curve="-90"/>
+<wire x1="182.72125" y1="37.62375" x2="183.67375" y2="37.62375" width="0.1524" layer="100"/>
+<wire x1="183.67375" y1="37.62375" x2="183.99125" y2="37.30625" width="0.1524" layer="100" curve="-90"/>
+<wire x1="183.99125" y1="37.30625" x2="183.99125" y2="22.5425" width="0.1524" layer="100"/>
+<wire x1="183.99125" y1="22.5425" x2="183.67375" y2="22.225" width="0.1524" layer="100" curve="-90"/>
+<wire x1="183.67375" y1="22.225" x2="182.72125" y2="22.225" width="0.1524" layer="100"/>
+<wire x1="182.72125" y1="22.225" x2="182.40375" y2="22.5425" width="0.1524" layer="100" curve="-90"/>
 </plain>
 <attributes>
@@
 </drawing>
 <compatibility>
+<note version="6.3" minversion="6.2.2" severity="warning">
+Since Version 6.2.2 text objects can contain more than one line,
+which will not be processed correctly with this version.
+</note>
 <note version="8.2" severity="warning">
 Since Version 8.2, EAGLE supports online libraries. The ids
