File: More/hardware/boards/HEGduinoV1/ESP32_ADC_HUB.sch (EAGLE design)
At the start: 14 parts, among them J1 RJ11-2L-B, U1 PINHD-1X10, U2 LP5907MFX-3.3/NOPB

Commit message: hegduino 1.1 brd
Other:
- note added: "FEATHER"
- note added: "LOLIN32"
Changed lines of the file:
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@@
 <plain>
 <text x="97.79" y="93.98" size="1.778" layer="95">OPTIONAL NOISE-CANCELLING LDO, CONNECT JUMPER IF NOT IN USE</text>
+<text x="87.63" y="52.07" size="1.778" layer="95">FEATHER</text>
+<text x="175.26" y="53.34" size="1.778" layer="95">LOLIN32</text>
 </plain>
 <instances>
