File: Software/hardware/boards/HEGduinoV1/ESP32_ADC_HUB.brd (EAGLE design)
At the start: 71.9 x 30 mm, 14 parts, among them J1 RJ11-2L-B, U1 PINHD-1X10, U2 LP5907MFX-3.3/NOPB

Commit message: tweaks and fixes, lower power consumption on LOLIN32, brd updates
Parts:
- removed SJ1: SOLDERJUMPERNC, headers:SJ_2S_SMALL
- added 5V_FEATHER, NO_LDO: (no value), jumper:SJ
Connections:
- new net 5VBAT: 5V_FEATHER.1, C1.1, C3.1, JP5.8, U2.1, U2.3
- net VANA: now also NO_LDO.2; no longer R1.1, R2.1, SJ1.2
- net VBAT: now also 5V_FEATHER.2, NO_LDO.1, R1.1, R2.1; no longer C1.1, C3.1, SJ1.1, U2.1, U2.3
Routing:
- net 5VBAT: track 0.00 -> 19.3 mm
- net VANA: track 65.4 -> 61.5 mm, vias 1 -> 2
- net VBAT: track 93.2 -> 95.2 mm, vias 2 -> 1
- added copper zone on layer 1, net GND
Other:
- board text added: "10uF"
- board text added: "1uF"
- board text added: "ADS1115 this side."
- board text added: "Connect for Huzzah32 Feather"
- board text added: "Optional, connect NO_LDO if not in use"
- board text removed: "ADS1115"
