File: Software/hardware/boards/HEGduinoV1/ESP32_ADC_HUB.sch (EAGLE design)
At the start: 14 parts, among them J1 RJ11-2L-B, U1 PINHD-1X10, U2 LP5907MFX-3.3/NOPB

Commit message: tweaks and fixes, lower power consumption on LOLIN32, brd updates
Parts:
- removed SJ1: SOLDERJUMPERNC, headers:SOLDERJUMPERNC
- added 5V_FEATHER, NO_LDO: (no value), jumper:SJ
Connections:
- new net 5VBAT: 5V_FEATHER.1, C1.1, C3.1, JP5.8, U2.EN, U2.IN
- net VANA: now also NO_LDO.2; no longer R1.1, R2.1, SJ1.2
- net VBAT: now also 5V_FEATHER.2, NO_LDO.1, R1.1, R2.1; no longer C1.1, C3.1, SJ1.1, U2.EN, U2.IN
